Commit message: Change physical properties from gold to aluminum

File: physics_block.urdf (robot description, URDF)
Before this commit: robot block_2, 1 links, 0 joints
Links:
- link block_2_base_link: mass 1.93 -> 0.27

Commit message: Changed mass to reflect aluminum

File: physics_block.urdf (robot description, URDF)
Before this commit: robot block_2, 1 links, 0 joints
Links:
- link block_2_base_link: mass 0.27 -> 2.7

Commit message: idk what i did here too 3am :))

File: physics_block.urdf (robot description, URDF)
Before this commit: robot block_2, 1 links, 0 joints
Links:
- link block_2_base_link: mass 2.7 -> 0.1

Commit message: Added friction

File: physics_block.urdf (robot description, URDF)
Before this commit: robot block_2, 1 links, 0 joints
Links:
- link block_2_base_link: mass 0.1 -> 7.85

Commit message: Changed physical properties to reflect 0.1^3 cast iron

File: physics_block.urdf (robot description, URDF)
Before this commit: robot block_2, 1 links, 0 joints
Links:
- link block_2_base_link: mass 7.85 -> 7.15

Commit message: Updated dynamics

File: physics_block.urdf (robot description, URDF)
Before this commit: robot block_2, 1 links, 0 joints
Links:
- link block_2_base_link: mass 7.15 -> 15.7660
